File: KiCAD_PIC16F887_RTC/PIC16F887_RTC.kicad_pcb (KiCad board)
At the start: 2 copper layers, 45 parts, among them IC2 DS1307, J1 BARREL_JACK, J2 ICD, Q1 2SA1013, Q2 2SA1013, Q3 2SA1013, Q4 2SA1013, SW1 SW_Push, SW2 SW_Push, SW6 SW_Push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

Commit message: Copper pour done
Routing:
- net GND: track 401.9 -> 409.1 mm
- net /SDA: track 49.9 -> 52.7 mm
- net /BUZZER: track 22.2 -> 23.3 mm
- added copper zone on B.Cu, net GND
Changed lines of the file:
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@@
   (general
     (links 99)
-    (no_connects 99)
-    (area 37.725 95.324999 150.875002 179.405001)
+    (no_connects 0)
+    (area 37.725 93.049999 153.250002 179.405001)
     (thickness 1.6)
-    (drawings 0)
-    (tracks 527)
+    (drawings 6)
+    (tracks 535)
     (zones 0)
     (modules 45)
@@
       (net 5 /OSC2))
   )
+  (gr_line (start 36.5 91) (end 38 91.1) (layer B.SilkS) (width 0.2))
+  (gr_line (start 36.5 93.9) (end 36.5 91) (layer B.SilkS) (width 0.2))
+  (gr_line (start 36.7 181.1) (end 36.5 93.9) (layer B.SilkS) (width 0.2))
+  (gr_line (start 156.1 180.9) (end 36.7 181.1) (layer B.SilkS) (width 0.2))
+  (gr_line (start 156.1 91.1) (end 156.1 180.9) (layer B.SilkS) (width 0.2))
+  (gr_line (start 38 91.1) (end 156.1 91.1) (layer B.SilkS) (width 0.2))
   (segment (start 47.025 172.975) (end 49.025 172.975) (width 1.2) (layer B.Cu) (net 1))
   (segment (start 49.025 172.975) (end 51.775 170.225) (width 1.2) (layer B.Cu) (net 1))
@@
   (segment (start 41.925 111) (end 43.65 112.725) (width 1) (layer B.Cu) (net 1))
   (segment (start 43.65 112.725) (end 43.65 127.825) (width 1) (layer B.Cu) (net 1))
+  (segment (start 101.2 100.6) (end 96.875 100.6) (width 1) (layer B.Cu) (net 2))
+  (segment (start 96.875 100.6) (end 96.85 100.625) (width 1) (layer B.Cu) (net 2))
+  (segment (start 64.175 131.825) (end 62.14 133.86) (width 1) (layer B.Cu) (net 2))
+  (segment (start 62.14 133.86) (end 62.115 133.86) (width 1) (layer B.Cu) (net 2))
   (segment (start 48.85 137.525) (end 49.649999 138.324999) (width 0.7) (layer B.Cu) (net 2))
   (segment (start 49.675 140.225) (end 49.675 154.05) (width 0.7) (layer B.Cu) (net 2))
@@
   (segment (start 70.81 165.46) (end 73.55 165.46) (width 0.7) (layer B.Cu) (net 6))
   (segment (start 73.55 165.46) (end 73.66 165.35) (width 0.7) (layer B.Cu) (net 6))
+  (segment (start 84.3 174.85) (end 87.04 174.85) (width 1) (layer B.Cu) (net 7))
+  (segment (start 87.04 174.85) (end 87.1 174.91) (width 1) (layer B.Cu) (net 7))
   (segment (start 70.09 149.1) (end 68.95863 149.1) (width 0.7) (layer B.Cu) (net 7))
   (segment (start 68.95863 149.1) (end 67.725 150.33363) (width 0.7) (layer B.Cu) (net 7))
@@
   (segment (start 48.85 111.675) (end 49.525 111) (width 1) (layer B.Cu) (net 49))
   (segment (start 49.525 111) (end 54.85 111) (width 1) (layer B.Cu) (net 49))
+  (segment (start 43.875 140.05) (end 42.775 140.05) (width 1) (layer B.Cu) (net 50))
+  (segment (start 42.775 140.05) (end 42.75 140.025) (width 1) (layer B.Cu) (net 50))
   (segment (start 52.6 123.7) (end 54.85 123.7) (width 1) (layer B.Cu) (net 50))
   (segment (start 51.325 124.975) (end 52.6 123.7) (width 1) (layer B.Cu) (net 50))
@@
   (segment (start 54.85 151.64) (end 58.314998 151.64) (width 0.7) (layer B.Cu) (net 58))
   (via (at 63.475 156.800002) (size 1.2) (drill 0.8) (layers F.Cu B.Cu) (net 58))
+  (zone (net 2) (net_name GND) (layer B.Cu) (hatch edge 0.508)
+    (connect_pads (clearance 0.7))
+    (min_thickness 0.254)
+    (fill yes (arc_segments 16) (thermal_gap 0.508) (thermal_bridge_width 0.508))
+    (polygon
+      (pts
+        (xy 38 93) (xy 38 178.9) (xy 38 180) (xy 44 180) (xy 68 180)
+        (xy 111 180) (xy 133.1 180) (xy 154.7 180) (xy 155 130) (xy 155 116.5)
+        (xy 155 106) (xy 155.1 105.2) (xy 155 93)
+      )
+    )
+  )
 )

Commit message: Added 4 mounting hole - No DRC
Parts:
- added REF**: Hole_2.2mm, Mounting_Holes:MountingHole_2.2mm_M2_DIN965_Pad, F.Cu at (151.5, 176.9)
- added REF**: Hole_2.2mm, Mounting_Holes:MountingHole_2.2mm_M2_DIN965_Pad, F.Cu at (151.5, 95.3)
- added REF**: Hole_2.2mm, Mounting_Holes:MountingHole_2.2mm_M2_DIN965_Pad, F.Cu at (40.3, 176.9)
- added REF**: Hole_2.2mm, Mounting_Holes:MountingHole_2.2mm_M2_DIN965_Pad, F.Cu at (40.3, 95.3)
Routing:
- net /RESET: track 63.4 -> 62.2 mm
Changed lines of the file:
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@@
     (links 99)
     (no_connects 0)
-    (area 37.725 93.049999 153.250002 179.405001)
+    (area 36.399999 90.899999 156.471429 181.375)
     (thickness 1.6)
     (drawings 6)
     (tracks 535)
     (zones 0)
-    (modules 45)
+    (modules 49)
     (nets 71)
   )
@@
   )
   (setup
-    (last_trace_width 1)
+    (last_trace_width 1.5)
     (user_trace_width 0.7)
     (user_trace_width 1)
@@
     (pad 2 thru_hole circle (at 2.44094 0) (size 1.39954 1.39954) (drill 0.8001) (layers *.Cu *.Mask F.SilkS)
       (net 5 /OSC2))
+  )
+  (module Mounting_Holes:MountingHole_2.2mm_M2_DIN965_Pad (layer F.Cu)
+    (at 151.5 176.9)
+    (descr "Mounting Hole 2.2mm, M2, DIN965")
+    (tags "mounting hole 2.2mm m2 din965")
+    (fp_text reference REF** (at 0 -2.9) (layer F.SilkS)
+      (effects (font (size 1 1) (thickness 0.15)))
+    )
+    (fp_text value Hole_2.2mm (at 0 2.9) (layer F.Fab)
+      (effects (font (size 1 1) (thickness 0.15)))
+    )
+    (fp_circle (center 0 0) (end 1.9 0) (layer Cmts.User) (width 0.15))
+    (fp_circle (center 0 0) (end 2.15 0) (layer F.CrtYd) (width 0.05))
+    (pad 1 thru_hole circle (at 0 0) (size 3.8 3.8) (drill 2.2) (layers *.Cu *.Mask))
+  )
+  (module Mounting_Holes:MountingHole_2.2mm_M2_DIN965_Pad (layer F.Cu)
+    (at 151.5 95.3)
+    (descr "Mounting Hole 2.2mm, M2, DIN965")
+    (tags "mounting hole 2.2mm m2 din965")
+    (fp_text reference REF** (at 0 -2.9) (layer F.SilkS)
+      (effects (font (size 1 1) (thickness 0.15)))
+    )
+    (fp_text value Hole_2.2mm (at 0 2.9) (layer F.Fab)
+      (effects (font (size 1 1) (thickness 0.15)))
+    )
+    (fp_circle (center 0 0) (end 1.9 0) (layer Cmts.User) (width 0.15))
+    (fp_circle (center 0 0) (end 2.15 0) (layer F.CrtYd) (width 0.05))
+    (pad 1 thru_hole circle (at 0 0) (size 3.8 3.8) (drill 2.2) (layers *.Cu *.Mask))
+  )
+  (module Mounting_Holes:MountingHole_2.2mm_M2_DIN965_Pad (layer F.Cu)
+    (at 40.3 176.9)
+    (descr "Mounting Hole 2.2mm, M2, DIN965")
+    (tags "mounting hole 2.2mm m2 din965")
+    (fp_text reference REF** (at 0 -2.9) (layer F.SilkS)
+      (effects (font (size 1 1) (thickness 0.15)))
+    )
+    (fp_text value Hole_2.2mm (at 8 2) (layer F.Fab)
+      (effects (font (size 1 1) (thickness 0.15)))
+    )
+    (fp_circle (center 0 0) (end 1.9 0) (layer Cmts.User) (width 0.15))
+    (fp_circle (center 0 0) (end 2.15 0) (layer F.CrtYd) (width 0.05))
+    (pad 1 thru_hole circle (at 0 0) (size 3.8 3.8) (drill 2.2) (layers *.Cu *.Mask))
+  )
+  (module Mounting_Holes:MountingHole_2.2mm_M2_DIN965_Pad (layer F.Cu)
+    (at 40.3 95.3)
+    (descr "Mounting Hole 2.2mm, M2, DIN965")
+    (tags "mounting hole 2.2mm m2 din965")
+    (fp_text reference REF** (at 0 -2.9) (layer F.SilkS)
+      (effects (font (size 1 1) (thickness 0.15)))
+    )
+    (fp_text value Hole_2.2mm (at 7 -1.6) (layer F.Fab)
+      (effects (font (size 1 1) (thickness 0.15)))
+    )
+    (fp_circle (center 0 0) (end 1.9 0) (layer Cmts.User) (width 0.15))
+    (fp_circle (center 0 0) (end 2.15 0) (layer F.CrtYd) (width 0.05))
+    (pad 1 thru_hole circle (at 0 0) (size 3.8 3.8) (drill 2.2) (layers *.Cu *.Mask))
   )
   (gr_line (start 36.5 91) (end 38 91.1) (layer B.SilkS) (width 0.2))
@@
   (segment (start 109.975 176.95) (end 110.95 175.975) (width 0.7) (layer B.Cu) (net 10))
   (segment (start 110.95 175.975) (end 110.95 173.85) (width 0.7) (layer B.Cu) (net 10))
+  (segment (start 76.14 104.395) (end 75.340001 103.595001) (width 0.7) (layer B.Cu) (net 12))
+  (segment (start 75.340001 103.595001) (end 68.245001 103.595001) (width 0.7) (layer B.Cu) (net 12))
+  (segment (start 68.245001 103.595001) (end 65.9 101.25) (width 0.7) (layer B.Cu) (net 12))
+  (segment (start 65.9 101.25) (end 65.9 97.525) (width 0.7) (layer B.Cu) (net 12))
+  (segment (start 65.9 97.525) (end 64.3 95.925) (width 0.7) (layer B.Cu) (net 12))
+  (segment (start 41.23 98.87) (end 41.23 99.25) (width 0.7) (layer B.Cu) (net 12))
+  (segment (start 64.3 95.925) (end 44.175 95.925) (width 0.7) (layer B.Cu) (net 12))
+  (segment (start 44.175 95.925) (end 41.23 98.87) (width 0.7) (layer B.Cu) (net 12))
   (segment (start 46.925 105.875) (end 41.7 105.875) (width 1) (layer F.Cu) (net 12))
   (segment (start 41.7 105.875) (end 41.675 105.85) (width 1) (layer F.Cu) (net 12))
@@
   (segment (start 46.97 105.92) (end 46.925 105.875) (width 1) (layer B.Cu) (net 12))
   (via (at 46.925 105.875) (size 1.2) (drill 0.8) (layers F.Cu B.Cu) (net 12))
-  (segment (start 76.14 104.395) (end 75.340001 103.595001) (width 0.7) (layer B.Cu) (net 12))
-  (segment (start 75.340001 103.595001) (end 68.245001 103.595001) (width 0.7) (layer B.Cu) (net 12))
-  (segment (start 41.23 96.82) (end 41.23 99.25) (width 0.7) (layer B.Cu) (net 12))
-  (segment (start 68.245001 103.595001) (end 65.9 101.25) (width 0.7) (layer B.Cu) (net 12))
-  (segment (start 65.9 101.25) (end 65.9 97.525) (width 0.7) (layer B.Cu) (net 12))
-  (segment (start 42.125 95.925) (end 41.23 96.82) (width 0.7) (layer B.Cu) (net 12))
-  (segment (start 65.9 97.525) (end 64.3 95.925) (width 0.7) (layer B.Cu) (net 12))
-  (segment (start 64.3 95.925) (end 42.125 95.925) (width 0.7) (layer B.Cu) (net 12))
   (segment (start 48.85 99.25) (end 48.85 97.925) (width 0.7) (layer B.Cu) (net 13))
   (segment (start 48.85 97.925) (end 49.625 97.15) (width 0.7) (layer B.Cu) (net 13))
@@
     (polygon
       (pts
-        (xy 38 93) (xy 38 178.9) (xy 38 180) (xy 44 180) (xy 68 180)
+        (xy 37 92) (xy 37 178.9) (xy 37 180) (xy 44 180) (xy 68 180)
         (xy 111 180) (xy 133.1 180) (xy 154.7 180) (xy 155 130) (xy 155 116.5)
-        (xy 155 106) (xy 155.1 105.2) (xy 155 93)
+        (xy 155 106) (xy 155.1 105.2) (xy 155 92)
       )
     )

Commit message: Test Circuit done, display Minute and sec
Other:
- board text added: "PIC16F887RTC_V1"
- board text added: "PMLUAN"
Changed lines of the file:
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@@
     (links 99)
     (no_connects 0)
-    (area 36.399999 90.899999 156.471429 181.375)
+    (area 36.399999 90.899999 156.471429 181.200001)
     (thickness 1.6)
-    (drawings 6)
+    (drawings 8)
     (tracks 535)
     (zones 0)
@@
     (visible_elements 7FFFFFFF)
     (pcbplotparams
-      (layerselection 0x00030_80000001)
+      (layerselection 0x00000_80000000)
       (usegerberextensions false)
       (excludeedgelayer true)
@@
       (padsonsilk false)
       (subtractmaskfromsilk false)
-      (outputformat 1)
+      (outputformat 4)
       (mirror false)
-      (drillshape 1)
+      (drillshape 0)
       (scaleselection 1)
-      (outputdirectory ""))
+      (outputdirectory Export/))
   )
   (net 0 "")
@@
     (pad 1 thru_hole circle (at 0 0) (size 3.8 3.8) (drill 2.2) (layers *.Cu *.Mask))
   )
+  (gr_text PIC16F887RTC_V1 (at 110.8 161.2) (layer B.Cu)
+    (effects (font (size 1.5 1.5) (thickness 0.3)) (justify mirror))
+  )
+  (gr_text PMLUAN (at 111.4 169.6) (layer B.Cu)
+    (effects (font (size 1.5 1.5) (thickness 0.3)) (justify mirror))
+  )
   (gr_line (start 36.5 91) (end 38 91.1) (layer B.SilkS) (width 0.2))
